File: FSR_to_can/FSR_to_can.kicad_sch (KiCad schematic)
At the start: 0 parts

Commit message: 0927_inLab
Parts:
- added U1: ATMEGA328P-AU, digikey-footprints:TQFP-32_7x7mm, symbol dk_Embedded-Microcontrollers:ATMEGA328P-AU
Connections:
- new net +5V: U1.18 (AVCC), U1.4 (VCC), U1.6 (VCC)
- new net GND: U1.21 (GND), U1.3 (GND), U1.5 (GND)

Commit message: 1st_ordered
Parts:
- added C1, C2: 0.1u, Capacitor_SMD:C_0805_2012Metric, symbol Device:C
- added C3, C4: 1u, Capacitor_SMD:C_0805_2012Metric, symbol Device:C
- added C5: 4.7u, Capacitor_SMD:C_0805_2012Metric, symbol Device:C_Polarized
- added C6: 10u, Capacitor_SMD:C_0805_2012Metric, symbol Device:C
- added C7: 22u, Capacitor_SMD:C_0805_2012Metric, symbol Device:C
- added C8: 0.1uF, Capacitor_SMD:C_0805_2012Metric, symbol Device:C
- added D1: SCK, LED_SMD:LED_0603_1608Metric_Pad1.05x0.95mm_HandSolder, symbol Device:LED
- added D2: power, LED_SMD:LED_0603_1608Metric_Pad1.05x0.95mm_HandSolder, symbol Device:LED
- added H1, H2, H3, H4: MountingHole, MountingHole:MountingHole_2.2mm_M2_ISO14580, symbol Mechanical:MountingHole
- added J1: FSR_socket, Connector_JST:JST_ZH_S5B-ZR-SM4A-TF_1x05-1MP_P1.50mm_Horizontal, symbol Connector:Conn_01x05_Socket
- added J2: write, Connector_JST:JST_ZH_B5B-ZR_1x05_P1.50mm_Vertical, symbol Connector:Conn_01x05_Socket
- added J3: boot, Connector_JST:JST_ZH_B6B-ZR_1x06_P1.50mm_Vertical, symbol Connector:Conn_01x06_Socket
- added J4: power_socket, Connector_JST:JST_XH_S2B-XH-A_1x02_P2.50mm_Horizontal, symbol Connector:Conn_01x02_Socket
- added J5: can_socket, Connector_JST:JST_ZH_S2B-ZR-SM4A-TF_1x02-1MP_P1.50mm_Horizontal, symbol Connector:Conn_01x02_Socket
- added JP1: Term, Jumper:SolderJumper-2_P1.3mm_Open_RoundedPad1.0x1.5mm, symbol Jumper:Jumper_2_Small_Open
- added R1, R2, R3, R4, R5, R6, R7: 1k, Resistor_SMD:R_0603_1608Metric, symbol Device:R_Small
- added R8: 120, Resistor_SMD:R_0603_1608Metric, symbol Device:R_Small
- added SW1: SW_Push, push_switch:TVAF06-A020B-R, symbol Switch:SW_Push
- added U2: AMS1117-5.0, Package_TO_SOT_SMD:SOT-223-3_TabPin2, symbol Regulator_Linear:AMS1117-5.0
- added U3: MCP2515-xST, Package_SO:TSSOP-20_4.4x6.5mm_P0.65mm, symbol Interface_CAN_LIN:MCP2515-xST
- added U4: MCP2561-E-SN, Package_SO:SOIC-8_3.9x4.9mm_P1.27mm, symbol Interface_CAN_LIN:MCP2561-E-SN
- added Y1: 16MHz, Crystal:Resonator_SMD_Murata_CSTxExxV-3Pin_3.0x1.1mm_HandSoldering, symbol Device:Crystal_GND2
- added Y2: 8MHz, Crystal:Resonator_SMD_Murata_CSTxExxV-3Pin_3.0x1.1mm_HandSoldering, symbol Device:Crystal_GND2
Connections:
- net +5V: now also C3.1, C4.1, C5.1, C7.1, C8.1, J2.1 (Pin_1), J3.1 (Pin_1), R1.1, R6.1, R7.2, U2.2 (VO), U3.19 (~{RESET}), U3.20 (VDD), U4.3 (VDD)
- net GND: now also C1.2, C3.2, C4.2, C5.2, C6.2, C7.2, C8.2, D1.1 (K), D2.1 (K), J1.1 (Pin_1), J2.2 (Pin_2), J3.2 (Pin_2), J4.1 (Pin_1), R2.2, SW1.1, U2.1 (GND), U3.10 (VSS), U4.2 (VSS), U4.8 (STBY), Y1.2, Y2.2
- net SS_atmega: now reaches U1.14 (PB2)
- net SS_atmega: now also U3.18 (~{CS})
- net MOSI_atmega: now reaches U1.15 (PB3)
- net MOSI_atmega: now also J3.4 (Pin_4), U3.16 (SI)
- net MISO_atmega: now reaches U1.16 (PB4)
- net MISO_atmega: now also J3.5 (Pin_5), U3.17 (SO)
- net SCK_atmega: now reaches U1.17 (PB5)
- net SCK_atmega: now also J3.6 (Pin_6), R5.2, U3.14 (SCK)
- net at U1.20 (AREF): now also C1.1
- net A1: now reaches U1.24 (PC1)
- net A2: now reaches U1.25 (PC2)
- net A3: now reaches U1.26 (PC3)
- net A4: now reaches U1.27 (PC4)
- net RESET: now reaches U1.29 (PC6)
- net RESET: now also C2.1, J3.3 (Pin_3), R6.2, SW1.2
- net at U1.30 (PD0): now also R3.1
- net at U1.31 (PD1): now also R4.1
- net INT: now reaches U1.32 (PD2)
- net INT: now also U3.13 (~{INT})
- net at U1.7 (PB6): now also Y1.3
- net at U1.8 (PB7): now also Y1.1
- new net: D1.2 (A), R5.1
- new net: JP1.2 (B), R8.2
- new net: U3.1 (TXCAN), U4.1 (TXD)
- new net: U3.2 (RXCAN), U4.4 (RXD)
- new net: U3.8 (OSC2), Y2.1
- new net: U3.9 (OSC1), Y2.3
- new net: D2.2 (A), R7.1
- new net +12V: C6.1, J4.2 (Pin_2), U2.3 (VI)
- new net CAN_N: J5.1 (Pin_1), JP1.1 (A), U4.6 (CANL)
- new net CAN_P: J5.2 (Pin_2), R8.1, U4.7 (CANH)
- new net DTR: C2.2, J2.5 (Pin_5)
- new net Dual_FSR_current/Vin_half: R1.2, R2.1
- new net FSR1: J1.2 (Pin_2)
- new net FSR2: J1.3 (Pin_3)
- new net FSR3: J1.4 (Pin_4)
- new net FSR4: J1.5 (Pin_5)
- new net RX: J2.3 (Pin_3), R3.2
- new net TX: J2.4 (Pin_4), R4.2
- no-connect marks 0 -> 18
Other:
- added sheet Dual_FSR_current (Dual_FSR_current.kicad_sch)
- added sheet Dual_FSR_current1 (Dual_FSR_current.kicad_sch)
