File: main_esp32e_can/DCDC_TPS62933_3V3.kicad_sch (KiCad schematic)
At the start: 9 parts, among them U4 TPS62933

Commit message: 1st_ordered
Parts:
- C13: renamed from C10; footprint (none) -> Capacitor_SMD:C_0805_2012Metric
- C14: renamed from C11; footprint (none) -> Capacitor_SMD:C_0805_2012Metric
- C15: renamed from C12; footprint (none) -> Capacitor_SMD:C_0805_2012Metric
- C16: renamed from C13; footprint (none) -> Capacitor_SMD:C_0805_2012Metric
- C17: renamed from C14; footprint (none) -> Capacitor_SMD:C_0805_2012Metric
- L2: renamed from L1; footprint (none) -> Inductor_SMD:L_Bourns-SRN8040_8x8.15mm
- R26: renamed from R13; footprint (none) -> Resistor_SMD:R_0603_1608Metric
- R27: renamed from R14; footprint (none) -> Resistor_SMD:R_0603_1608Metric
- renumbered U4 to U10
Connections:
- net 3V3out: now reaches C16.2, L2.1, U10.5 (SW)
Changed lines of the file:
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@@
+		)
+	)
+	(label "3V3out"
+		(at 152.4 86.36 0)
+		(effects
+			(font
+				(size 1.27 1.27)
+			)
+			(justify left bottom)
 		)
 	)
@@
 		(dnp no)
 		(fields_autoplaced yes)
-		(property "Reference" "C13"
+		(property "Reference" "C16"
 			(at 158.75 81.2799 0)
 			(effects
@@
 			)
 		)
-		(property "Footprint" ""
+		(property "Footprint" "Capacitor_SMD:C_0805_2012Metric"
 			(at 155.9052 86.36 0)
 			(effects
@@
 			(project ""
 				(path "/c0f075e2-5381-4409-948d-59a846480f0e/62be41a3-d98d-4b28-a1b7-23dd5fce8c3c/31129f53-636f-4212-bd0f-f9cec8397b4f"
-					(reference "C13")
+					(reference "C16")
 					(unit 1)
 				)
@@
 		(dnp no)
 		(fields_autoplaced yes)
-		(property "Reference" "U4"
+		(property "Reference" "U10"
 			(at 140.97 71.12 0)
 			(effects
@@
 			(project ""
 				(path "/c0f075e2-5381-4409-948d-59a846480f0e/62be41a3-d98d-4b28-a1b7-23dd5fce8c3c/31129f53-636f-4212-bd0f-f9cec8397b4f"
-					(reference "U4")
+					(reference "U10")
 					(unit 1)
 				)
@@
 		(dnp no)
 		(fields_autoplaced yes)
-		(property "Reference" "R13"
+		(property "Reference" "R26"
 			(at 177.8 90.1699 0)
 			(effects
@@
 			)
 		)
-		(property "Footprint" ""
+		(property "Footprint" "Resistor_SMD:R_0603_1608Metric"
 			(at 173.482 91.44 90)
 			(effects
@@
 			(project ""
 				(path "/c0f075e2-5381-4409-948d-59a846480f0e/62be41a3-d98d-4b28-a1b7-23dd5fce8c3c/31129f53-636f-4212-bd0f-f9cec8397b4f"
-					(reference "R13")
+					(reference "R26")
 					(unit 1)
 				)
@@
 		(dnp no)
 		(fields_autoplaced yes)
-		(property "Reference" "C12"
+		(property "Reference" "C15"
 			(at 123.19 81.28 90)
 			(effects
@@
 			)
 		)
-		(property "Footprint" ""
+		(property "Footprint" "Capacitor_SMD:C_0805_2012Metric"
 			(at 127 87.9348 0)
 			(effects
@@
 			(project "main_esp32e_can"
 				(path "/c0f075e2-5381-4409-948d-59a846480f0e/62be41a3-d98d-4b28-a1b7-23dd5fce8c3c/31129f53-636f-4212-bd0f-f9cec8397b4f"
-					(reference "C12")
+					(reference "C15")
 					(unit 1)
 				)
@@
 		(dnp no)
 		(fields_autoplaced yes)
-		(property "Reference" "L1"
+		(property "Reference" "L2"
 			(at 166.37 81.28 90)
 			(effects
@@
 			)
 		)
-		(property "Footprint" ""
+		(property "Footprint" "Inductor_SMD:L_Bourns-SRN8040_8x8.15mm"
 			(at 166.37 86.36 0)
 			(effects
@@
 			(project ""
 				(path "/c0f075e2-5381-4409-948d-59a846480f0e/62be41a3-d98d-4b28-a1b7-23dd5fce8c3c/31129f53-636f-4212-bd0f-f9cec8397b4f"
-					(reference "L1")
+					(reference "L2")
 					(unit 1)
 				)
@@
 		(dnp no)
 		(fields_autoplaced yes)
-		(property "Reference" "R14"
+		(property "Reference" "R27"
 			(at 177.8 100.3299 0)
 			(effects
@@
 			)
 		)
-		(property "Footprint" ""
+		(property "Footprint" "Resistor_SMD:R_0603_1608Metric"
 			(at 173.482 101.6 90)
 			(effects
@@
 			(project "main_esp32e_can"
 				(path "/c0f075e2-5381-4409-948d-59a846480f0e/62be41a3-d98d-4b28-a1b7-23dd5fce8c3c/31129f53-636f-4212-bd0f-f9cec8397b4f"
-					(reference "R14")
+					(reference "R27")
 					(unit 1)
 				)
@@
 		(dnp no)
 		(fields_autoplaced yes)
-		(property "Reference" "C10"
+		(property "Reference" "C13"
 			(at 101.6 82.5499 0)
 			(effects
@@
 			)
 		)
-		(property "Footprint" ""
+		(property "Footprint" "Capacitor_SMD:C_0805_2012Metric"
 			(at 98.7552 87.63 0)
 			(effects
@@
 			(project "main_esp32e_can"
 				(path "/c0f075e2-5381-4409-948d-59a846480f0e/62be41a3-d98d-4b28-a1b7-23dd5fce8c3c/31129f53-636f-4212-bd0f-f9cec8397b4f"
-					(reference "C10")
+					(reference "C13")
 					(unit 1)
 				)
@@
 		(dnp no)
 		(fields_autoplaced yes)
-		(property "Reference" "C14"
+		(property "Reference" "C17"
 			(at 190.5 90.1699 0)
 			(effects
@@
 			)
 		)
-		(property "Footprint" ""
+		(property "Footprint" "Capacitor_SMD:C_0805_2012Metric"
 			(at 187.6552 95.25 0)
 			(effects
@@
 			(project "main_esp32e_can"
 				(path "/c0f075e2-5381-4409-948d-59a846480f0e/62be41a3-d98d-4b28-a1b7-23dd5fce8c3c/31129f53-636f-4212-bd0f-f9cec8397b4f"
-					(reference "C14")
+					(reference "C17")
 					(unit 1)
 				)
@@
 		(dnp no)
 		(fields_autoplaced yes)
-		(property "Reference" "C11"
+		(property "Reference" "C14"
 			(at 115.57 82.5499 0)
 			(effects
@@
 			)
 		)
-		(property "Footprint" ""
+		(property "Footprint" "Capacitor_SMD:C_0805_2012Metric"
 			(at 112.7252 87.63 0)
 			(effects
@@
 			(project "main_esp32e_can"
 				(path "/c0f075e2-5381-4409-948d-59a846480f0e/62be41a3-d98d-4b28-a1b7-23dd5fce8c3c/31129f53-636f-4212-bd0f-f9cec8397b4f"
-					(reference "C11")
-					(unit 1)
-				)
+					(reference "C14")
+					(unit 1)
+				)
