File: main_esp32e_can/DCDC_TPS62933_7V4.kicad_sch (KiCad schematic)
At the start: 9 parts, among them U5 TPS62933

Commit message: 1st_ordered
Parts:
- C18: renamed from C15; footprint (none) -> Capacitor_SMD:C_0805_2012Metric
- C19: renamed from C16; footprint (none) -> Capacitor_SMD:C_0805_2012Metric
- C20: renamed from C17; footprint (none) -> Capacitor_SMD:C_0805_2012Metric
- C21: renamed from C18; footprint (none) -> Capacitor_SMD:C_0805_2012Metric
- C22: renamed from C19; footprint (none) -> Capacitor_SMD:C_0805_2012Metric
- L3: renamed from L2; footprint (none) -> Inductor_SMD:L_Bourns-SRN8040_8x8.15mm
- R28: renamed from R15; footprint (none) -> Resistor_SMD:R_0603_1608Metric
- R29: renamed from R16; footprint (none) -> Resistor_SMD:R_0603_1608Metric
- renumbered U5 to U11
Connections:
- net 7.4Vout: now reaches C21.2, L3.1, U11.5 (SW)
Changed lines of the file:
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@@
 	(paper "A4")
+	(junction
+		(at 158.75 86.36)
+		(diameter 0)
+		(color 0 0 0 0)
+	)
 	(junction
 		(at 186.69 86.36)
@@
 	(wire
 		(pts
+			(xy 158.75 86.36) (xy 162.56 86.36)
+		)
+		(stroke
+			(width 0)
+			(type default)
+		)
+	)
+	(wire
+		(pts
 			(xy 186.69 86.36) (xy 198.12 86.36)
 		)
@@
 	(wire
 		(pts
-			(xy 154.94 86.36) (xy 162.56 86.36)
+			(xy 154.94 86.36) (xy 158.75 86.36)
 		)
 		(stroke
@@
 	(wire
 		(pts
+			(xy 158.75 88.9) (xy 158.75 86.36)
+		)
+		(stroke
+			(width 0)
+			(type default)
+		)
+	)
+	(wire
+		(pts
 			(xy 111.76 78.74) (xy 111.76 80.01)
 		)
@@
 			(width 0)
 			(type default)
+		)
+	)
+	(label "7.4Vout"
+		(at 158.75 88.9 180)
+		(effects
+			(font
+				(size 1.27 1.27)
+			)
+			(justify right bottom)
 		)
 	)
@@
 		(dnp no)
 		(fields_autoplaced yes)
-		(property "Reference" "C15"
+		(property "Reference" "C18"
 			(at 101.6 82.5499 0)
 			(effects
@@
 			)
 		)
-		(property "Footprint" ""
+		(property "Footprint" "Capacitor_SMD:C_0805_2012Metric"
 			(at 98.7552 87.63 0)
 			(effects
@@
 			(project "main_esp32e_can"
 				(path "/c0f075e2-5381-4409-948d-59a846480f0e/62be41a3-d98d-4b28-a1b7-23dd5fce8c3c/da8501cc-4ef0-4247-8e76-1779f540fa5a"
-					(reference "C15")
+					(reference "C18")
 					(unit 1)
 				)
@@
 		(dnp no)
 		(fields_autoplaced yes)
-		(property "Reference" "R15"
+		(property "Reference" "R28"
 			(at 177.8 90.1699 0)
 			(effects
@@
 			)
 		)
-		(property "Footprint" ""
+		(property "Footprint" "Resistor_SMD:R_0603_1608Metric"
 			(at 173.482 91.44 90)
 			(effects
@@
 				)
 				(path "/c0f075e2-5381-4409-948d-59a846480f0e/62be41a3-d98d-4b28-a1b7-23dd5fce8c3c/da8501cc-4ef0-4247-8e76-1779f540fa5a"
-					(reference "R15")
+					(reference "R28")
 					(unit 1)
 				)
@@
 		(dnp no)
 		(fields_autoplaced yes)
-		(property "Reference" "C18"
+		(property "Reference" "C21"
 			(at 158.75 81.2799 0)
 			(effects
@@
 			)
 		)
-		(property "Footprint" ""
+		(property "Footprint" "Capacitor_SMD:C_0805_2012Metric"
 			(at 155.9052 86.36 0)
 			(effects
@@
 				)
 				(path "/c0f075e2-5381-4409-948d-59a846480f0e/62be41a3-d98d-4b28-a1b7-23dd5fce8c3c/da8501cc-4ef0-4247-8e76-1779f540fa5a"
-					(reference "C18")
+					(reference "C21")
 					(unit 1)
 				)
@@
 		(dnp no)
 		(fields_autoplaced yes)
-		(property "Reference" "R16"
+		(property "Reference" "R29"
 			(at 177.8 100.3299 0)
 			(effects
@@
 			)
 		)
-		(property "Footprint" ""
+		(property "Footprint" "Resistor_SMD:R_0603_1608Metric"
 			(at 173.482 101.6 90)
 			(effects
@@
 			(project "main_esp32e_can"
 				(path "/c0f075e2-5381-4409-948d-59a846480f0e/62be41a3-d98d-4b28-a1b7-23dd5fce8c3c/da8501cc-4ef0-4247-8e76-1779f540fa5a"
-					(reference "R16")
+					(reference "R29")
 					(unit 1)
 				)
@@
 		(dnp no)
 		(fields_autoplaced yes)
-		(property "Reference" "L2"
+		(property "Reference" "L3"
 			(at 166.37 81.28 90)
 			(effects
@@
 			)
 		)
-		(property "Footprint" ""
+		(property "Footprint" "Inductor_SMD:L_Bourns-SRN8040_8x8.15mm"
 			(at 166.37 86.36 0)
 			(effects
@@
 				)
 				(path "/c0f075e2-5381-4409-948d-59a846480f0e/62be41a3-d98d-4b28-a1b7-23dd5fce8c3c/da8501cc-4ef0-4247-8e76-1779f540fa5a"
-					(reference "L2")
+					(reference "L3")
 					(unit 1)
 				)
@@
 		(dnp no)
 		(fields_autoplaced yes)
-		(property "Reference" "C17"
+		(property "Reference" "C20"
 			(at 123.19 81.28 90)
 			(effects
@@
 			)
 		)
-		(property "Footprint" ""
+		(property "Footprint" "Capacitor_SMD:C_0805_2012Metric"
 			(at 127 87.9348 0)
 			(effects
@@
 			(project "main_esp32e_can"
 				(path "/c0f075e2-5381-4409-948d-59a846480f0e/62be41a3-d98d-4b28-a1b7-23dd5fce8c3c/da8501cc-4ef0-4247-8e76-1779f540fa5a"
-					(reference "C17")
+					(reference "C20")
 					(unit 1)
 				)
@@
 		(dnp no)
 		(fields_autoplaced yes)
-		(property "Reference" "C16"
+		(property "Reference" "C19"
 			(at 115.57 82.5499 0)
 			(effects
@@
 			)
 		)
-		(property "Footprint" ""
+		(property "Footprint" "Capacitor_SMD:C_0805_2012Metric"
 			(at 112.7252 87.63 0)
 			(effects
@@
 			(project "main_esp32e_can"
 				(path "/c0f075e2-5381-4409-948d-59a846480f0e/62be41a3-d98d-4b28-a1b7-23dd5fce8c3c/da8501cc-4ef0-4247-8e76-1779f540fa5a"
-					(reference "C16")
+					(reference "C19")
 					(unit 1)
 				)
@@
 		(dnp no)
 		(fields_autoplaced yes)
-		(property "Reference" "U5"
+		(property "Reference" "U11"
 			(at 140.97 71.12 0)
 			(effects
@@
 				)
 				(path "/c0f075e2-5381-4409-948d-59a846480f0e/62be41a3-d98d-4b28-a1b7-23dd5fce8c3c/da8501cc-4ef0-4247-8e76-1779f540fa5a"
-					(reference "U5")
+					(reference "U11")
 					(unit 1)
 				)
@@
 		(dnp no)
 		(fields_autoplaced yes)
-		(property "Reference" "C19"
+		(property "Reference" "C22"
 			(at 190.5 90.1699 0)
 			(effects
@@
 			)
 		)
-		(property "Footprint" ""
+		(property "Footprint" "Capacitor_SMD:C_0805_2012Metric"
 			(at 187.6552 95.25 0)
 			(effects
@@
 			(project "main_esp32e_can"
 				(path "/c0f075e2-5381-4409-948d-59a846480f0e/62be41a3-d98d-4b28-a1b7-23dd5fce8c3c/da8501cc-4ef0-4247-8e76-1779f540fa5a"
-					(reference "C19")
-					(unit 1)
-				)
+					(reference "C22")
+					(unit 1)
+				)
