File: main_esp32e_can/Level_Shifter.kicad_sch (KiCad schematic)
At the start: 3 parts

Commit message: 0928_inhouse
Parts:
- renumbered Q to Q5, R6 to R10, R to R9
Changed lines of the file:
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@@
 		(dnp no)
 		(fields_autoplaced yes)
-		(property "Reference" "Q"
+		(property "Reference" "Q5"
 			(at 137.16 105.41 90)
 			(effects
@@
 		(instances
 			(project "main_esp32e_can"
+				(path "/c0f075e2-5381-4409-948d-59a846480f0e/1a165a23-a96a-44e6-9976-953fe6ccf7ae"
+					(reference "Q8")
+					(unit 1)
+				)
+				(path "/c0f075e2-5381-4409-948d-59a846480f0e/481fd7a4-f3b8-4924-b85d-7a964c819d37"
+					(reference "Q5")
+					(unit 1)
+				)
 				(path "/c0f075e2-5381-4409-948d-59a846480f0e/7fabc5d7-0f02-4149-95a1-fa513e825ccf"
 					(reference "Q6")
+					(unit 1)
+				)
+				(path "/c0f075e2-5381-4409-948d-59a846480f0e/ae448462-19a4-47c2-a78b-0a1ef408c5af"
+					(reference "Q7")
 					(unit 1)
 				)
@@
 		(dnp no)
 		(fields_autoplaced yes)
-		(property "Reference" "R"
+		(property "Reference" "R9"
 			(at 129.54 90.1699 0)
 			(effects
@@
 		(instances
 			(project "main_esp32e_can"
+				(path "/c0f075e2-5381-4409-948d-59a846480f0e/1a165a23-a96a-44e6-9976-953fe6ccf7ae"
+					(reference "R21")
+					(unit 1)
+				)
+				(path "/c0f075e2-5381-4409-948d-59a846480f0e/481fd7a4-f3b8-4924-b85d-7a964c819d37"
+					(reference "R9")
+					(unit 1)
+				)
 				(path "/c0f075e2-5381-4409-948d-59a846480f0e/7fabc5d7-0f02-4149-95a1-fa513e825ccf"
-					(reference "R10")
+					(reference "R11")
+					(unit 1)
+				)
+				(path "/c0f075e2-5381-4409-948d-59a846480f0e/ae448462-19a4-47c2-a78b-0a1ef408c5af"
+					(reference "R19")
 					(unit 1)
 				)
@@
 		(dnp no)
 		(fields_autoplaced yes)
-		(property "Reference" "R6"
+		(property "Reference" "R10"
 			(at 149.86 90.1699 0)
 			(effects
@@
 		(instances
 			(project "main_esp32e_can"
+				(path "/c0f075e2-5381-4409-948d-59a846480f0e/1a165a23-a96a-44e6-9976-953fe6ccf7ae"
+					(reference "R22")
+					(unit 1)
+				)
 				(path "/c0f075e2-5381-4409-948d-59a846480f0e/481fd7a4-f3b8-4924-b85d-7a964c819d37"
-					(reference "R6")
+					(reference "R10")
 					(unit 1)
 				)
 				(path "/c0f075e2-5381-4409-948d-59a846480f0e/7fabc5d7-0f02-4149-95a1-fa513e825ccf"
-					(reference "R11")
-					(unit 1)
-				)
+					(reference "R12")
+					(unit 1)
+				)
+				(path "/c0f075e2-5381-4409-948d-59a846480f0e/ae448462-19a4-47c2-a78b-0a1ef408c5af"
+					(reference "R20")
+					(unit 1)
+				)

Commit message: 1st_ordered
Parts:
- removed Q5: 2N7002K, Package_TO_SOT_SMD:SOT-23, symbol Transistor_FET:2N7002K
- added Q8: 2N7002K, Package_TO_SOT_SMD:SOT-23, symbol Transistor_FET:2N7002K
- R22: renamed from R9; footprint (none) -> Resistor_SMD:R_0603_1608Metric
- R23: renamed from R10; footprint (none) -> Resistor_SMD:R_0603_1608Metric
Connections:
- net Hsig: now also Q8.3 (D)
- net LV: now also Q8.1 (G)
- net Lsig: now also Q8.2 (S)
Changed lines of the file:
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@@
 		(dnp no)
 		(fields_autoplaced yes)
-		(property "Reference" "Q5"
+		(property "Reference" "Q8"
 			(at 137.16 105.41 90)
 			(effects
@@
 			)
 		)
+		(pin "1"
+		)
 		(pin "2"
 		)
 		(pin "3"
 		)
-		(pin "1"
-		)
 		(instances
-			(project "main_esp32e_can"
-				(path "/c0f075e2-5381-4409-948d-59a846480f0e/1a165a23-a96a-44e6-9976-953fe6ccf7ae"
+			(project ""
+				(path "/c0f075e2-5381-4409-948d-59a846480f0e/481fd7a4-f3b8-4924-b85d-7a964c819d37"
 					(reference "Q8")
 					(unit 1)
 				)
-				(path "/c0f075e2-5381-4409-948d-59a846480f0e/481fd7a4-f3b8-4924-b85d-7a964c819d37"
-					(reference "Q5")
-					(unit 1)
-				)
 				(path "/c0f075e2-5381-4409-948d-59a846480f0e/7fabc5d7-0f02-4149-95a1-fa513e825ccf"
-					(reference "Q6")
+					(reference "Q9")
 					(unit 1)
 				)
 				(path "/c0f075e2-5381-4409-948d-59a846480f0e/ae448462-19a4-47c2-a78b-0a1ef408c5af"
-					(reference "Q7")
+					(reference "Q10")
 					(unit 1)
 				)
@@
 		(dnp no)
 		(fields_autoplaced yes)
-		(property "Reference" "R9"
+		(property "Reference" "R22"
 			(at 129.54 90.1699 0)
 			(effects
@@
 			)
 		)
-		(property "Footprint" ""
+		(property "Footprint" "Resistor_SMD:R_0603_1608Metric"
 			(at 125.222 91.44 90)
 			(effects
@@
 		(instances
 			(project "main_esp32e_can"
-				(path "/c0f075e2-5381-4409-948d-59a846480f0e/1a165a23-a96a-44e6-9976-953fe6ccf7ae"
-					(reference "R21")
-					(unit 1)
-				)
 				(path "/c0f075e2-5381-4409-948d-59a846480f0e/481fd7a4-f3b8-4924-b85d-7a964c819d37"
-					(reference "R9")
+					(reference "R22")
 					(unit 1)
 				)
 				(path "/c0f075e2-5381-4409-948d-59a846480f0e/7fabc5d7-0f02-4149-95a1-fa513e825ccf"
-					(reference "R11")
+					(reference "R24")
 					(unit 1)
 				)
 				(path "/c0f075e2-5381-4409-948d-59a846480f0e/ae448462-19a4-47c2-a78b-0a1ef408c5af"
-					(reference "R19")
+					(reference "R30")
 					(unit 1)
 				)
@@
 		(dnp no)
 		(fields_autoplaced yes)
-		(property "Reference" "R10"
+		(property "Reference" "R23"
 			(at 149.86 90.1699 0)
 			(effects
@@
 			)
 		)
-		(property "Footprint" ""
+		(property "Footprint" "Resistor_SMD:R_0603_1608Metric"
 			(at 145.542 91.44 90)
 			(effects
@@
 		(instances
 			(project "main_esp32e_can"
-				(path "/c0f075e2-5381-4409-948d-59a846480f0e/1a165a23-a96a-44e6-9976-953fe6ccf7ae"
-					(reference "R22")
-					(unit 1)
-				)
 				(path "/c0f075e2-5381-4409-948d-59a846480f0e/481fd7a4-f3b8-4924-b85d-7a964c819d37"
-					(reference "R10")
+					(reference "R23")
 					(unit 1)
 				)
 				(path "/c0f075e2-5381-4409-948d-59a846480f0e/7fabc5d7-0f02-4149-95a1-fa513e825ccf"
-					(reference "R12")
+					(reference "R25")
 					(unit 1)
 				)
 				(path "/c0f075e2-5381-4409-948d-59a846480f0e/ae448462-19a4-47c2-a78b-0a1ef408c5af"
-					(reference "R20")
-					(unit 1)
-				)
+					(reference "R31")
+					(unit 1)
+				)
