File: main_esp32e_can/main_esp32e_can.kicad_sch (KiCad schematic)
At the start: 0 parts

Commit message: 0927_inLab
Parts:
- added C3, C5, C6, C7: 0.1u, symbol Device:C
- added C4: 22u, symbol Device:C
- added J4: write_socket, symbol Connector:Conn_01x06_Socket
- added J5: can_socket, symbol Connector:Conn_01x02_Socket
- added JP1: Termination_R, symbol Jumper:Jumper_2_Open
- added Q4, Q5: 2SC2712, symbol Transistor_BJT:Q_NPN_BEC
- added R12: 120, symbol Device:R
- added R7, R8, R9: 10k, symbol Device:R
- added SW1: RESET, symbol Switch:SW_Push
- added SW2: BOOT, symbol Switch:SW_Push
- added U1: ESP32-WROOM-32E, RF_Module:ESP32-WROOM-32D, symbol RF_Module:ESP32-WROOM-32E
- added U2: MCP2561-E-SN, Package_SO:SOIC-8_3.9x4.9mm_P1.27mm, symbol Interface_CAN_LIN:MCP2561-E-SN
Connections:
- new net: J5.2 (Pin_2), R12.2, U2.6 (CANL)
- new net: J5.1 (Pin_1), JP1.2 (B), U2.7 (CANH)
- new net: JP1.1 (A), R12.1
- new net: Q4.1 (B), R9.2
- new net: Q5.1 (B), R8.2
- new net +3.3V: C3.1, C4.1, C5.1, C6.1, J4.1 (Pin_1), Q4.3 (C), R7.1, R7.2, SW1.2, U1.2 (VDD), U1.3 (EN)
- new net +5V: U2.3 (VDD)
- new net DTR: J4.5 (Pin_5), Q5.2 (E), R9.1
- new net GND: C3.2, C4.2, C5.2, C6.2, C7.2, J4.2 (Pin_2), SW1.1, SW2.1, U1.1 (GND), U1.15 (GND), U1.38 (GND), U1.39 (GND), U2.2 (VSS), U2.8 (STBY)
- new net IO0: C7.1, Q5.3 (C), SW2.2, U1.25 (IO0)
- new net Level_Shifter/Hsig: U2.1 (TXD)
- new net Level_Shifter1/Hsig: U2.4 (RXD)
- new net RTS: J4.6 (Pin_6), Q4.2 (E), R8.1
- new net RXD: J4.3 (Pin_3), U1.35 (TXD0/IO1)
- new net TXD: J4.4 (Pin_4), U1.34 (RXD0/IO3)
- no-connect marks 0 -> 3
Other:
- added sheet Level_Shifter (Level_Shifter.kicad_sch)
- added sheet Level_Shifter1 (Level_Shifter.kicad_sch)
- added sheet power_supply (power_supply.kicad_sch)

Commit message: 0928_inhouse
Parts:
- added J10, J11, J12, J13: ICS_socket, symbol Connector:Conn_01x03_Socket
- added J14, J15: 12Vout, symbol Connector:Conn_01x02_Socket
- added J8, J9: ICS_socket_7V4, symbol Connector:Conn_01x03_Socket
- added R17, R18: 2k, symbol Device:R
- added U6: ~, symbol MyLib:BNO055_Module
- added U7: 74LVC2G241, symbol 74xGxx:74LVC2G241
- renumbered C4 to C1, C5 to C2, C6 to C4, C7 to C5, J4 to J1, J5 to J2, Q4 to Q1, Q5 to Q2, R7 to R1, R9 to R2, R8 to R3, R12 to R4
Connections:
- net +3.3V: now also R17.1, R18.2, U6.1 (Vin)
- net +5V: now also U7.8 (VCC)
- net CRX: now also U1.12 (IO27)
- net CTX: now also U1.11 (IO26)
- net GND: now also U6.2 (GND), U6.7 (GND), U7.4 (GND)
- net EN_TTL: now reaches U1.24 (IO2)
- net EN_TTL: now also U7.1, U7.7
- net RX2: now reaches U1.27 (IO16)
- net TX2: now reaches U1.28 (IO17)
- net SDA: now reaches U1.33 (IO21)
- net SDA: now also R18.1, U6.3 (SDA/T)
- net SCL: now reaches U1.36 (IO22)
- net SCL: now also R17.2, U6.4 (SCL/R)
- new net +12V: J10.2 (Pin_2), J11.2 (Pin_2), J12.2 (Pin_2), J13.2 (Pin_2), J14.2 (Pin_2), J15.2 (Pin_2)
- new net +7.5V: J8.2 (Pin_2), J9.2 (Pin_2)
- new net GND1: J10.1 (Pin_1), J11.1 (Pin_1), J12.1 (Pin_1), J13.1 (Pin_1), J14.1 (Pin_1), J15.1 (Pin_1), J8.1 (Pin_1), J9.1 (Pin_1)
- new net ICS_sig: J10.3 (Pin_3), J11.3 (Pin_3), J12.3 (Pin_3), J13.3 (Pin_3), J8.3 (Pin_3), J9.3 (Pin_3), U7.2, U7.3
- new net Level_Shifter2/Hsig: U7.6
- new net Level_Shifter3/Hsig: U7.5
- no-connect marks 3 -> 20
Other:
- added sheet Level_Shifter2 (Level_Shifter.kicad_sch)
- added sheet Level_Shifter3 (Level_Shifter.kicad_sch)
- moved on the sheet: J2, JP1, R4, U2

Commit message: 1st_ordered
Parts:
- added C6: 0.1u, Capacitor_SMD:C_0805_2012Metric, symbol Device:C
- added H1, H2, H3, H4: MountingHole, MountingHole:MountingHole_3.2mm_M3, symbol Mechanical:MountingHole
- added J9: can_socket, Connector_JST:JST_ZH_B2B-ZR_1x02_P1.50mm_Vertical, symbol Connector:Conn_01x02_Socket
- added Q1, Q2, Q5: 2N7002K, Package_TO_SOT_SMD:SOT-23, symbol Transistor_FET:2N7002K
- added R11, R12, R6: 350, Resistor_SMD:R_0603_1608Metric, symbol Device:R_Small
- added R13, R4, R7: 120, Resistor_SMD:R_0603_1608Metric, symbol Device:R_Small
- added R14, R5, R8: 1k, Resistor_SMD:R_0603_1608Metric, symbol Device:R_Small
- added U3, U4, U5: TLP2361_TPL_E, digikey-footprints:SOIC-6-5_W4.55mm, symbol dk_Optoisolators-Logic-Output:TLP2361_TPL_E
- C1, C2, C3, C4, C5: footprint (none) -> Capacitor_SMD:C_0805_2012Metric
- J1: footprint (none) -> Connector_JST:JST_ZH_B6B-ZR_1x06_P1.50mm_Vertical
- J10: renamed from J14; footprint (none) -> Connector_JST:JST_XA_B02B-XASK-1_1x02_P2.50mm_Vertical
- J11: renamed from J15; footprint (none) -> Connector_JST:JST_XA_B02B-XASK-1_1x02_P2.50mm_Vertical
- J2: renamed from J10; footprint (none) -> Connector_JST:JST_ZH_B3B-ZR_1x03_P1.50mm_Vertical
- J3: renamed from J11; footprint (none) -> Connector_JST:JST_ZH_B3B-ZR_1x03_P1.50mm_Vertical
- J4: renamed from J12; footprint (none) -> Connector_JST:JST_ZH_B3B-ZR_1x03_P1.50mm_Vertical
- J5: renamed from J13; footprint (none) -> Connector_JST:JST_ZH_B3B-ZR_1x03_P1.50mm_Vertical
- J6: renamed from J8; footprint (none) -> Connector_JST:JST_ZH_B3B-ZR_1x03_P1.50mm_Vertical
- J7: renamed from J9; footprint (none) -> Connector_JST:JST_ZH_B3B-ZR_1x03_P1.50mm_Vertical
- J8: renamed from J2; footprint (none) -> Connector_JST:JST_ZH_B2B-ZR_1x02_P1.50mm_Vertical
- JP1: value Termination_R -> Term; footprint (none) -> Jumper:SolderJumper-2_P1.3mm_Open_RoundedPad1.0x1.5mm
- Q3: renamed from Q1; footprint (none) -> Package_TO_SOT_SMD:SOT-23
- Q4: renamed from Q2; footprint (none) -> Package_TO_SOT_SMD:SOT-23
- R1: footprint (none) -> Resistor_SMD:R_0603_1608Metric
- R10: renamed from R3; footprint (none) -> Resistor_SMD:R_0603_1608Metric
- R15: renamed from R4; footprint (none) -> Resistor_SMD:R_0603_1608Metric
- R2: renamed from R18; footprint (none) -> Resistor_SMD:R_0603_1608Metric
- R3: renamed from R17; footprint (none) -> Resistor_SMD:R_0603_1608Metric
- R9: renamed from R2; footprint (none) -> Resistor_SMD:R_0603_1608Metric
- SW1, SW2: footprint (none) -> Button_Switch_SMD:SW_SPST_B3S-1000
- U1: renamed from U6; value ~ -> BNO055_module; footprint (none) -> myfootprint:BNO055_module
- U6: renamed from U7; footprint (none) -> Package_SO:VSSOP-8_2.3x2mm_P0.5mm
- renumbered U1 to U2, U2 to U7
Connections:
- net +12V: no longer J10.2 (Pin_2), J11.2 (Pin_2)
- net +3.3V: no longer C2.1, C4.1, Q3.3 (C), R1.2, SW1.2, U2.3 (EN)
- net +5V: now also C6.1, R11.1, R6.1, U4.6 (VCC); no longer U6.8 (VCC)
- net EN_TTL: now also R4.1; no longer U6.1, U6.7
- net GND: now also J10.1 (Pin_1), J11.1 (Pin_1), C6.2, Q1.2 (S), Q2.2 (S), R5.2, R8.2, U4.4 (GND); no longer U6.4 (GND)
- net GND1: now also U6.4 (GND), Q5.2 (S), R14.2, U3.4 (GND), U5.4 (GND); no longer J10.1 (Pin_1), J11.1 (Pin_1)
- net Level_Shifter2/Hsig: now also U4.5 (VO); no longer U6.6
- net TX2: now also R7.1
- net CAN_N: now reaches R15.2, U7.6 (CANL)
- net CAN_N: now also J8.1 (Pin_1), J9.1 (Pin_1); no longer J8.2 (Pin_2)
- net CAN_P: now reaches JP1.2 (B), U7.7 (CANH)
- net CAN_P: now also J8.2 (Pin_2), J9.2 (Pin_2); no longer J8.1 (Pin_1)
- net Level_Shifter3/Hsig: no longer names the net of U6.5
- net Level_Shifter3/Hsig: now also U5.5 (VO)
- new net: Q5.1 (G), R13.2, R14.1
- new net: Q5.3 (D), U4.3
- new net: U3.5 (VO), U6.1, U6.7
- new net: R13.1, U6.6
- new net: Q2.1 (G), R7.2, R8.1
- new net: Q2.3 (D), U5.3
- new net: R11.2, U5.1
- new net: Q1.1 (G), R4.2, R5.1
- new net: R12.2, U4.1
- new net: R6.2, U3.1
- new net: Q1.3 (D), U3.3
- new net +12VA: J10.2 (Pin_2), J11.2 (Pin_2)
- new net +5VA: R12.1, U3.6 (VCC), U5.6 (VCC), U6.8 (VCC)
- new net EN: C2.1, C4.1, Q3.3 (C), R1.2, SW1.2, U2.3 (EN)
Other:
- removed sheet Level_Shifter3
- moved on the sheet: J10, J11, J2, J3, J4, J5, J6, J7, J8, JP1, R15, U6A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
