File: main_esp32e_can/power_supply.kicad_sch (KiCad schematic)
At the start: 11 parts, among them J1 Batt_socket, J2 SW_strong, J3 SW_logic, Q1 TK100E06N1, Q2 TK100E06N1

Commit message: 0928_inhouse
Parts:
- removed Q1, Q2: TK100E06N1, symbol Transistor_FET:Q_NMOS_GDS
- added C8: 10u, symbol Device:C_Polarized
- added C9: 22u, symbol Device:C_Polarized
- added D1: LED_motor, symbol Device:LED
- added D2: LED_logic, symbol Device:LED
- added J6: LED_strong, Connector_AMASS:AMASS_XT60-F_1x02_P7.20mm_Vertical, symbol Connector:Conn_01x02_Socket
- added J7: LED_logic, Connector_AMASS:AMASS_XT60-F_1x02_P7.20mm_Vertical, symbol Connector:Conn_01x02_Socket
- added L3: CM2021Y330R, symbol Device:L_Coupled_1423
- added Q3, Q4: TJ60S04M3L, symbol Transistor_FET:Q_PMOS_GDS
- added R23, R24: R, symbol Device:R
- added U3: AMS1117-5.0, Package_TO_SOT_SMD:SOT-223-3_TabPin2, symbol Regulator_Linear:AMS1117-5.0
- C6: renamed from C2; value C_Polarized -> 100u
- C7: renamed from C1; value C_Polarized -> 470u
- renumbered J1 to J3, J2 to J4, J3 to J5, R2 to R5, R1 to R6, R3 to R7, R4 to R8
Connections:
- net GND1 is gone; now on net -BATT: C7.2
- net +12V: now also Q3.3 (S), R23.1; no longer C6.1, J3.2 (Pin_2), J4.1 (Pin_1), J5.1 (Pin_1)
- net -BATT: now also J4.1 (Pin_1), D1.1 (K), J6.2 (Pin_2), L3.2; no longer R6.2, R8.2
- net GND: now also J5.1 (Pin_1), C8.2, C9.2, D2.1 (K), J7.2 (Pin_2), L3.3, U3.1 (GND)
- net at R7.2, R8.1: now also Q4.1 (G)
- net at R5.2, R6.1: now also Q3.1 (G)
- new net: D1.2 (A), R23.2
- new net: D2.2 (A), R24.2
- new net +5V: C9.1, R24.1, U3.2 (VO)
- new net +BATT: J3.2 (Pin_2), J6.1 (Pin_1), J7.1 (Pin_1), L3.1, Q3.2 (D), R6.2
- new net DCDC_TPS62933_3V3/Vin: C6.1, C8.1, Q4.3 (S), U3.3 (VI)
- new net logic+: L3.4, Q4.2 (D), R8.2
Other:
- added sheet DCDC_TPS62933_3V3 (DCDC_TPS62933_3V3.kicad_sch)
- added sheet DCDC_TPS62933_7V4 (DCDC_TPS62933_7V4.kicad_sch)
- moved on the sheet: C6, C7, J3, J4, J5, R5, R6, R7, R8

Commit message: 1st_ordered
Parts:
- added C8: 0.33u, Capacitor_SMD:C_0805_2012Metric, symbol Device:C
- added C9: 0.1u, Capacitor_SMD:C_0805_2012Metric, symbol Device:C
- added U8: L78L05_SOT89, Package_TO_SOT_SMD:SOT-89-3, symbol Regulator_Linear:L78L05_SOT89
- C10: renamed from C6; footprint (none) -> Capacitor_SMD:CP_Elec_6.3x5.9
- C11: renamed from C8; footprint (none) -> Capacitor_SMD:CP_Elec_5x5.8
- C12: renamed from C9; footprint (none) -> Capacitor_SMD:CP_Elec_6.3x5.9
- C7: footprint (none) -> Capacitor_SMD:CP_Elec_10x12.6
- D1, D2: footprint (none) -> Capacitor_SMD:C_0603_1608Metric
- J12: renamed from J3; footprint Connector_AMASS:AMASS_XT60-F_1x02_P7.20mm_Vertical -> Connector_AMASS:AMASS_XT60-M_1x02_P7.20mm_Vertical
- J13: renamed from J4; footprint Connector_AMASS:AMASS_XT60-F_1x02_P7.20mm_Vertical -> Connector_JST:JST_XA_B02B-XASK-1-A_1x02_P2.50mm_Vertical
- J14: renamed from J6; footprint Connector_AMASS:AMASS_XT60-F_1x02_P7.20mm_Vertical -> Connector_JST:JST_XH_B2B-XH-AM_1x02_P2.50mm_Vertical
- J15: renamed from J7; footprint Connector_AMASS:AMASS_XT60-F_1x02_P7.20mm_Vertical -> Connector_JST:JST_XH_B2B-XH-AM_1x02_P2.50mm_Vertical
- J16: renamed from J5; footprint Connector_AMASS:AMASS_XT60-F_1x02_P7.20mm_Vertical -> Connector_JST:JST_XA_B02B-XASK-1-A_1x02_P2.50mm_Vertical
- L1: renamed from L3; footprint (none) -> myfootprint:CM2021Y330R
- Q6: renamed from Q3; footprint (none) -> Package_TO_SOT_SMD:TO-252-2
- Q7: renamed from Q4; footprint (none) -> Package_TO_SOT_SMD:TO-252-2
- R16: renamed from R6; value 1K -> 10k; footprint (none) -> Resistor_SMD:R_0603_1608Metric
- R17: renamed from R5; footprint (none) -> Resistor_SMD:R_0603_1608Metric
- R18: renamed from R23; value R -> 2k; footprint (none) -> Resistor_SMD:R_0603_1608Metric
- R19: renamed from R24; value R -> 1k; footprint (none) -> Resistor_SMD:R_0603_1608Metric
- R20: renamed from R8; value 1K -> 10k; footprint (none) -> Resistor_SMD:R_0603_1608Metric
- R21: renamed from R7; footprint (none) -> Resistor_SMD:R_0603_1608Metric
- renumbered U3 to U9
Connections:
- net +12V: now also J14.1 (Pin_1), C8.1, U8.3 (IN)
- net +BATT: no longer J14.1 (Pin_1), J15.1 (Pin_1)
- net -BATT renamed GND1
- net GND1: now also C8.2, C9.2, U8.2 (GND)
- net DCDC_TPS62933_3V3/Vin renamed +12VA
- net +12VA: now also J15.1 (Pin_1)
- new net +5VA: C9.1, U8.1 (OUT)
Other:
- moved on the sheet: D1, D2, J14, R18, R19
